File: schematics/1600WRMS-MATRIX-1.4-III-CLASS-H-AUDIO-POWER-AMPLIFIER-NS-LAB-VERSION/1600WRMS-MATRIX-1.4-III-CLASS-H-AUDIO-POWER-AMPLIFIER-NS-LAB-VERSION.sch (KiCad schematic (older format))
At the start: 262 parts, among them Q301 2N5551, Q401 2N5551, Q402 2N5551, Q403 2N5401, Q404 2N5401, Q405 2N5551, Q406 MJE340, Q407 2N5401, Q408 MJE350, Q409 MJE350, Q410 MJE340, Q501 2N5401, Q502 MJE350, Q503 2N5551, Q504 MJE340, Q505 MJE340, Q506 MJE15032, Q507 2SC5200, Q5081 2SC5200, Q50810 2SC5200, Q50811 2SC5200, Q5082 2SC5200, Q5083 2SC5200, Q5084 2SC5200, Q5085 2SC5200, Q5086 2SC5200, Q5087 2SC5200, Q5088 2SC5200, Q5089 2SC5200, Q509 MJE15033, Q510 2SA1943, Q511 2SA1943, Q5111 2SA1943, Q51110 2SA1943, Q51111 2SA1943, Q5113 2SA1943, Q5114 2SA1943, Q5115 2SA1943, Q5116 2SA1943, Q5117 2SA1943, Q5118 2SA1943, Q5119 2SA1943, Q512 2N5551, Q513 2N5401, Q601 2N5551, Q602 2N5401, Q603 2N5401, Q604 2N5401, Q605 2N5551, Q606 2N5551, Q701 2N5551, Q702 2N5401, Q703 2N5551, Q704 2N5551, Q705 TIP42C, X6011 IRF9540, X6012 IRF9540, X6021 IRF540, X6022 IRF540

Commit message: Commit Thu May  9 01:23:26 UTC 2019
Parts:
- C404, C405: value 390pF -> 120pF
Changed lines of the file:
@@
 $Descr A3 16535 11693
 encoding utf-8
-Sheet 2 2
+Sheet 1 1
 Title "1600W RMS Class-H Audio Power Amplifier Core Circuit"
 Date "2019-05-08"
@@
 AR Path="/5CE6421B/5CF0C4E5" Ref="Q?"  Part="1"
 AR Path="/5C87359F/5CF0C4E5" Ref="Q401"  Part="1"
+AR Path="/5CF0C4E5" Ref="Q401"  Part="1"
 F 0 "Q401" H 2700 2300 50  0000 C CNN
 F 1 "2N5551" H 2700 2200 50  0000 C CNN
@@
 AR Path="/5CE6421B/5CF0C4EF" Ref="Q?"  Part="1"
 AR Path="/5C87359F/5CF0C4EF" Ref="Q402"  Part="1"
+AR Path="/5CF0C4EF" Ref="Q402"  Part="1"
 F 0 "Q402" H 3000 2300 50  0000 C CNN
 F 1 "2N5551" H 3000 2200 50  0000 C CNN
@@
 AR Path="/5CE6421B/5CF0C501" Ref="Q?"  Part="1"
 AR Path="/5C87359F/5CF0C501" Ref="Q406"  Part="1"
+AR Path="/5CF0C501" Ref="Q406"  Part="1"
 F 0 "Q406" H 3400 2850 50  0000 C CNN
 F 1 "MJE340" H 3400 2750 50  0000 C CNN
@@
 AR Path="/5CE6421B/5CF0C50B" Ref="Q?"  Part="1"
 AR Path="/5C87359F/5CF0C50B" Ref="Q405"  Part="1"
+AR Path="/5CF0C50B" Ref="Q405"  Part="1"
 F 0 "Q405" H 3100 3050 50  0000 C CNN
 F 1 "2N5551" H 3100 2950 50  0000 C CNN
@@
 AR Path="/5CE6421B/5CF0C517" Ref="#GND?"  Part="1"
 AR Path="/5C87359F/5CF0C517" Ref="#GND0136"  Part="1"
+AR Path="/5CF0C517" Ref="#GND0136"  Part="1"
 F 0 "#GND0136" H 2500 3100 50  0001 C CNN
 F 1 "0" H 2500 3287 50  0001 C CNN
@@
 AR Path="/5CE6421B/5CF0C52D" Ref="Q?"  Part="1"
 AR Path="/5C87359F/5CF0C52D" Ref="Q409"  Part="1"
+AR Path="/5CF0C52D" Ref="Q409"  Part="1"
 F 0 "Q409" H 4550 1650 50  0000 C CNN
 F 1 "MJE350" H 4550 1750 50  0000 C CNN
@@
 AR Path="/5CE6421B/5CF0C547" Ref="Q?"  Part="1"
 AR Path="/5C87359F/5CF0C547" Ref="Q408"  Part="1"
+AR Path="/5CF0C547" Ref="Q408"  Part="1"
 F 0 "Q408" H 3400 5150 50  0000 C CNN
 F 1 "MJE350" H 3400 5250 50  0000 C CNN
@@
 AR Path="/5CE6421B/5CF0C553" Ref="#GND?"  Part="1"
 AR Path="/5C87359F/5CF0C553" Ref="#GND0137"  Part="1"
+AR Path="/5CF0C553" Ref="#GND0137"  Part="1"
 F 0 "#GND0137" H 2500 5350 50  0001 C CNN
 F 1 "0" H 2500 5537 50  0001 C CNN
@@
 AR Path="/5CE6421B/5CF0C565" Ref="Q?"  Part="1"
 AR Path="/5C87359F/5CF0C565" Ref="Q403"  Part="1"
+AR Path="/5CF0C565" Ref="Q403"  Part="1"
 F 0 "Q403" H 2750 5650 50  0000 C CNN
 F 1 "2N5401" H 2750 5750 50  0000 C CNN
@@
 AR Path="/5CE6421B/5CF0C56F" Ref="Q?"  Part="1"
 AR Path="/5C87359F/5CF0C56F" Ref="Q410"  Part="1"
+AR Path="/5CF0C56F" Ref="Q410"  Part="1"
 F 0 "Q410" H 4550 6350 50  0000 C CNN
 F 1 "MJE340" H 4550 6250 50  0000 C CNN
@@
 AR Path="/5CE6421B/5CF0C5B6" Ref="C?"  Part="1"
 AR Path="/5C87359F/5CF0C5B6" Ref="C405"  Part="1"
+AR Path="/5CF0C5B6" Ref="C405"  Part="1"
 F 0 "C405" V 4550 6100 50  0000 C CNN
-F 1 "390pF" V 4450 6100 50  0000 C CNN
+F 1 "120pF" V 4450 6100 50  0000 C CNN
 F 2 "MATRIX_1.4:CAPACITOR_CERAMIC_STD" H 4200 6100 50  0001 C CNN
 F 3 "" H 4200 6100 50  0001 C CNN
@@
 AR Path="/5CE6421B/5CF0C5EB" Ref="R?"  Part="1"
 AR Path="/5C87359F/5CF0C5EB" Ref="R408"  Part="1"
+AR Path="/5CF0C5EB" Ref="R408"  Part="1"
 F 0 "R408" V 2900 2800 50  0000 C CNN
 F 1 "22k" V 2800 2900 50  0000 C CNN
@@
 AR Path="/5CE6421B/5CF0C5F2" Ref="R?"  Part="1"
 AR Path="/5C87359F/5CF0C5F2" Ref="R411"  Part="1"
+AR Path="/5CF0C5F2" Ref="R411"  Part="1"
 F 0 "R411" V 2600 5200 50  0000 C CNN
 F 1 "22k" V 2500 5200 50  0000 C CNN
@@
 AR Path="/5CE6421B/5CF0C5F8" Ref="R?"  Part="1"
 AR Path="/5C87359F/5CF0C5F8" Ref="R4141"  Part="1"
+AR Path="/5CF0C5F8" Ref="R4141"  Part="1"
 F 0 "R4141" H 4050 6750 50  0000 L CNN
 F 1 "150" H 4050 6650 50  0000 L CNN
@@
 AR Path="/5CE6421B/5CF0C616" Ref="R?"  Part="1"
 AR Path="/5C87359F/5CF0C616" Ref="R4131"  Part="1"
+AR Path="/5CF0C616" Ref="R4131"  Part="1"
 F 0 "R4131" H 4050 1350 50  0000 L CNN
 F 1 "150" H 4050 1250 50  0000 L CNN
@@
 AR Path="/5CE6421B/5CF0C61C" Ref="R?"  Part="1"
 AR Path="/5C87359F/5CF0C61C" Ref="R4091"  Part="1"
+AR Path="/5CF0C61C" Ref="R4091"  Part="1"
 F 0 "R4091" H 3250 3250 50  0000 L CNN
 F 1 "150" H 3250 3150 50  0000 L CNN
@@
 AR Path="/5CE6421B/5CF0C622" Ref="R?"  Part="1"
 AR Path="/5C87359F/5CF0C622" Ref="R4121"  Part="1"
+AR Path="/5CF0C622" Ref="R4121"  Part="1"
 F 0 "R4121" H 3250 4850 50  0000 L CNN
 F 1 "150" H 3250 4750 50  0000 L CNN
@@
 AR Path="/5CE6421B/5CF0C632" Ref="R?"  Part="1"
 AR Path="/5C87359F/5CF0C632" Ref="R406"  Part="1"
+AR Path="/5CF0C632" Ref="R406"  Part="1"
 F 0 "R406" H 3100 6750 50  0000 L CNN
 F 1 "470" H 3100 6650 50  0000 L CNN
@@
 AR Path="/5CE6421B/5CF0C638" Ref="R?"  Part="1"
 AR Path="/5C87359F/5CF0C638" Ref="R405"  Part="1"
+AR Path="/5CF0C638" Ref="R405"  Part="1"
 F 0 "R405" H 3100 1350 50  0000 L CNN
 F 1 "470" H 3100 1250 50  0000 L CNN
@@
 AR Path="/5CE6421B/5CF0C63E" Ref="R?"  Part="1"
 AR Path="/5C87359F/5CF0C63E" Ref="R4092"  Part="1"
+AR Path="/5CF0C63E" Ref="R4092"  Part="1"
 F 0 "R4092" H 3600 3250 50  0000 L CNN
 F 1 "680" H 3600 3150 50  0000 L CNN
@@
 AR Path="/5CE6421B/5CF0C644" Ref="R?"  Part="1"
 AR Path="/5C87359F/5CF0C644" Ref="R4122"  Part="1"
+AR Path="/5CF0C644" Ref="R4122"  Part="1"
 F 0 "R4122" H 3600 4850 50  0000 L CNN
 F 1 "680" H 3600 4750 50  0000 L CNN
@@
 AR Path="/5CE6421B/5CF0C64A" Ref="R?"  Part="1"
 AR Path="/5C87359F/5CF0C64A" Ref="R4142"  Part="1"
+AR Path="/5CF0C64A" Ref="R4142"  Part="1"
 F 0 "R4142" H 4400 6750 50  0000 L CNN
 F 1 "750" H 4400 6650 50  0000 L CNN
@@
 AR Path="/5CE6421B/5CF0C650" Ref="R?"  Part="1"
 AR Path="/5C87359F/5CF0C650" Ref="R4132"  Part="1"
+AR Path="/5CF0C650" Ref="R4132"  Part="1"
 F 0 "R4132" H 4400 1350 50  0000 L CNN
 F 1 "750" H 4400 1250 50  0000 L CNN
@@
 AR Path="/5CE6421B/5CF0C657" Ref="C?"  Part="1"
 AR Path="/5C87359F/5CF0C657" Ref="C404"  Part="1"
+AR Path="/5CF0C657" Ref="C404"  Part="1"
 F 0 "C404" V 4050 1900 50  0000 C CNN
-F 1 "390pF" V 3950 1900 50  0000 C CNN
+F 1 "120pF" V 3950 1900 50  0000 C CNN
 F 2 "MATRIX_1.4:CAPACITOR_CERAMIC_STD" H 4200 1900 50  0001 C CNN
 F 3 "" H 4200 1900 50  0001 C CNN
@@
 AR Path="/5CE6421B/5CF0C668" Ref="R?"  Part="1"
 AR Path="/5C87359F/5CF0C668" Ref="R407"  Part="1"
+AR Path="/5CF0C668" Ref="R407"  Part="1"
 F 0 "R407" H 3250 2500 50  0000 L CNN
 F 1 "270" H 3250 2400 50  0000 L CNN
@@
 AR Path="/5CE6421B/5CF0C672" Ref="Q?"  Part="1"
 AR Path="/5C87359F/5CF0C672" Ref="Q404"  Part="1"
+AR Path="/5CF0C672" Ref="Q404"  Part="1"
 F 0 "Q404" H 3050 5650 50  0000 C CNN
 F 1 "2N5401" H 3050 5750 50  0000 C CNN
@@
 AR Path="/5CE6421B/5CF0C679" Ref="R?"  Part="1"
 AR Path="/5C87359F/5CF0C679" Ref="R410"  Part="1"
+AR Path="/5CF0C679" Ref="R410"  Part="1"
 F 0 "R410" H 3250 5600 50  0000 L CNN
 F 1 "270" H 3250 5500 50  0000 L CNN
@@
 AR Path="/5CE6421B/5CF0C69E" Ref="Q?"  Part="1"
 AR Path="/5C87359F/5CF0C69E" Ref="Q407"  Part="1"
+AR Path="/5CF0C69E" Ref="Q407"  Part="1"
 F 0 "Q407" H 3100 4950 50  0000 C CNN
 F 1 "2N5401" H 3100 5050 50  0000 C CNN

Commit message: Commit Thu May  9 10:32:49 UTC 2019
Parts:
- added R305: 100k, MATRIX_1.4:RESISTOR_AXIAL_0.5W, symbol MATRIX_1.4:RESISTOR
- added R310: 2.7k, MATRIX_1.4:RESISTOR_AXIAL_0.25W, symbol MATRIX_1.4:RESISTOR
- C302: value 220uF -> 10uF
- D301, D302: value 1N4730 -> 1N4734; Spice_Model 1N4730 -> 1N4734
- R4012, R4042: value 150k -> 2.0
- renumbered R305 to R309, R309 to R311, R310 to R312, R311 to R313, R312 to R314
Connections:
- net 0: now also R310.2
- net M_OUT_RAW: now also R305.1
- net at C402.2, Q401.2 (B), Q403.2 (B)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: no longer R4011.2
- net at R4041.1, R4042.1: no longer C403.1
- net at C401.2, R4011.1: no longer R4012.1
- net at Q402.2 (B), Q404.2 (B), R403.2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: no longer R4042.2
- net at R309.2, XU302.3 (+): now also R310.1; no longer R306.1, XU302.5 (+)
- new net: C403.1, R4042.2
- new net: R305.2, R306.1, XU302.5 (+)
- new net: R4011.2, R4012.1
Other:
- note added: "S.O.A OUT: 80.8V RMS\n4-OHMS MAX. LOAD"
- note removed: "S.O.A OUT: 81.6V RMS\n4-OHMS MAX. LOAD"
- moved on the sheet: D301, R307, R311, R4041, XU302A
