File: schematics/1600WRMS-MATRIX-1.4-III-CLASS-H-AUDIO-POWER-AMPLIFIER-NS-LAB-VERSION/1600WRMS-MATRIX-1.4-III-CLASS-H-AUDIO-POWER-AMPLIFIER-NS-LAB-VERSION.sch (KiCad schematic (older format))
At the start: 264 parts, among them Q301 2N5551, Q401 2N5551, Q402 2N5551, Q403 2N5401, Q404 2N5401, Q405 2N5551, Q406 MJE340, Q407 2N5401, Q408 MJE350, Q409 MJE350, Q410 MJE340, Q501 2N5401, Q502 MJE350, Q503 2N5551, Q504 MJE340, Q505 MJE340, Q506 MJE15032, Q507 2SC5200, Q5081 2SC5200, Q50810 2SC5200, Q50811 2SC5200, Q5082 2SC5200, Q5083 2SC5200, Q5084 2SC5200, Q5085 2SC5200, Q5086 2SC5200, Q5087 2SC5200, Q5088 2SC5200, Q5089 2SC5200, Q509 MJE15033, Q510 2SA1943, Q511 2SA1943, Q5111 2SA1943, Q51110 2SA1943, Q51111 2SA1943, Q5113 2SA1943, Q5114 2SA1943, Q5115 2SA1943, Q5116 2SA1943, Q5117 2SA1943, Q5118 2SA1943, Q5119 2SA1943, Q512 2N5551, Q513 2N5401, Q601 2N5551, Q602 2N5401, Q603 2N5401, Q604 2N5401, Q605 2N5551, Q606 2N5551, Q701 2N5551, Q702 2N5401, Q703 2N5551, Q704 2N5551, Q705 TIP42C, X6011 IRF9540, X6012 IRF9540, X6021 IRF540, X6022 IRF540

Commit message: Commit Thu May  9 11:45:40 UTC 2019
Parts:
- C302: value 10uF -> 220uF
Changed lines of the file:
@@
 EESchema Schematic File Version 4
+LIBS:1600WRMS-MATRIX-1.4-III-CLASS-H-AUDIO-POWER-AMPLIFIER-NS-LAB-VERSION-cache
 EELAYER 29 0
 EELAYER END
@@
 P 7250 8850
 F 0 "C302" H 7450 8950 50  0000 C CNN
-F 1 "10uF" H 7450 8850 50  0000 C CNN
+F 1 "220uF" H 7450 8850 50  0000 C CNN
 F 2 "MATRIX_1.4:CAPACITOR_AE_D10mm" H 7250 8850 50  0001 C CNN
 F 3 "" H 7250 8850 50  0001 C CNN

Commit message: Commit Mon May 13 03:44:39 UTC 2019
Parts:
- R605, R614: footprint MATRIX_1.4:RESISTOR_AXIAL_0.25W -> MATRIX_1.4:RESISTOR_AXIAL_0.5W; Wattage (none) -> 0.5W
- X6011, X6012, X6021, X6022: footprint MATRIX_1.4:TO-220 -> MATRIX_1.4:TO-220-MIRRORED
- renumbered Q511 to Q5112
Changed lines of the file:
@@
 Sheet 1 1
 Title "1600W RMS Class-H Audio Power Amplifier Core Circuit"
-Date "2019-05-08"
+Date "2019-05-13"
 Rev ""
 Comp "Notice: LIMITER & F/S.O.C.P are courtesy of VCGA (https://github.com/vcga/vcga)"
@@
 Wire Wire Line
 	11750 1750 13050 1750
-Wire Wire Line
-	11750 1400 11750 1750
 Connection ~ 13050 1450
 Wire Wire Line
@@
 	8600 5450 8650 5450
 $Comp
-L MATRIX_1.4:Q_PNP Q511
+L MATRIX_1.4:Q_PNP Q5112
 U 1 1 5F01047B
 P 8800 5450
-F 0 "Q511" H 8550 5150 50  0000 C CNN
+F 0 "Q5112" H 8550 5150 50  0000 C CNN
 F 1 "2SA1943" H 8550 5250 50  0000 C CNN
 F 2 "MATRIX_1.4:TO-264-MIRRORED" H 8800 5450 50  0001 C CNN
@@
 F 0 "X6022" H 13700 6500 50  0000 L CNN
 F 1 "IRF540" H 13700 6400 50  0000 L CNN
-F 2 "MATRIX_1.4:TO-220" H 14450 6600 50  0001 C CNN
+F 2 "MATRIX_1.4:TO-220-MIRRORED" H 14450 6600 50  0001 C CNN
 F 3 "" H 14000 6750 50  0001 C CNN
 F 4 "X" H 15000 6700 50  0001 C CNN "Spice_Primitive"
@@
 Wire Wire Line
 	11150 6850 11150 6950
-Wire Wire Line
-	11150 1150 11150 1200
-Connection ~ 11150 1150
 Connection ~ 11150 1750
-Wire Wire Line
-	11150 1050 11150 1150
 Connection ~ 11150 1050
 Wire Wire Line
@@
 Wire Wire Line
 	11150 1750 11750 1750
-Wire Wire Line
-	11450 1150 11450 1450
-Wire Wire Line
-	11450 1450 11850 1450
-Wire Wire Line
-	11150 1150 11450 1150
 $Comp
 L MATRIX_1.4:DIODE D509
@@
 F 0 "X6021" H 13600 7050 50  0000 L CNN
 F 1 "IRF540" H 13600 6950 50  0000 L CNN
-F 2 "MATRIX_1.4:TO-220" H 14000 6600 50  0001 C CNN
+F 2 "MATRIX_1.4:TO-220-MIRRORED" H 14000 6600 50  0001 C CNN
 F 3 "" H 13550 6750 50  0001 C CNN
 F 4 "X" H 14550 6700 50  0001 C CNN "Spice_Primitive"
@@
 $EndComp
 $Comp
-L MATRIX_1.4:RESISTOR R614
-U 1 1 5E782811
-P 11750 6750
-F 0 "R614" H 11500 6800 50  0000 L CNN
-F 1 "68k" H 11500 6700 50  0000 L CNN
-F 2 "MATRIX_1.4:RESISTOR_AXIAL_0.25W" H 11750 6750 50  0001 C CNN
-F 3 "" H 11750 6750 50  0001 C CNN
-	1    11750 6750
-	1    0    0    -1
-$EndComp
-$Comp
 L MATRIX_1.4:RESISTOR R606
 U 1 1 5DE6083E
@@
 $EndComp
 $Comp
-L MATRIX_1.4:RESISTOR R605
-U 1 1 5DE38666
-P 11750 1250
-F 0 "R605" H 11500 1300 50  0000 L CNN
-F 1 "68k" H 11500 1200 50  0000 L CNN
-F 2 "MATRIX_1.4:RESISTOR_AXIAL_0.25W" H 11750 1250 50  0001 C CNN
-F 3 "" H 11750 1250 50  0001 C CNN
-	1    11750 1250
-	1    0    0    -1
-$EndComp
-$Comp
 L MATRIX_1.4:RESISTOR R604
 U 1 1 5DDD849C
@@
 F 0 "X6011" H 13600 1450 50  0000 L CNN
 F 1 "IRF9540" H 13600 1550 50  0000 L CNN
-F 2 "MATRIX_1.4:TO-220" H 14000 1100 50  0001 C CNN
+F 2 "MATRIX_1.4:TO-220-MIRRORED" H 14000 1100 50  0001 C CNN
 F 3 "" H 13550 1250 50  0001 C CNN
 F 4 "X" H 14550 1200 50  0001 C CNN "Spice_Primitive"
@@
 F 0 "X6012" H 13700 900 50  0000 L CNN
 F 1 "IRF9540" H 13650 1000 50  0000 L CNN
-F 2 "MATRIX_1.4:TO-220" H 14450 1100 50  0001 C CNN
+F 2 "MATRIX_1.4:TO-220-MIRRORED" H 14450 1100 50  0001 C CNN
 F 3 "" H 14000 1250 50  0001 C CNN
 F 4 "X" H 15000 1200 50  0001 C CNN "Spice_Primitive"
@@
 Wire Wire Line
 	2400 3600 2200 3600
+Wire Wire Line
+	11150 1050 11150 1150
+Wire Wire Line
+	11350 1450 11350 1150
+Wire Wire Line
+	11350 1150 11150 1150
+Connection ~ 11150 1150
+Wire Wire Line
+	11150 1150 11150 1200
+Wire Wire Line
+	11350 1450 11850 1450
+Wire Wire Line
+	11750 1400 11750 1750
+$Comp
+L MATRIX_1.4:RESISTOR R605
+U 1 1 5CEC619F
+P 11750 1250
+F 0 "R605" H 11600 1350 50  0000 C CNN
+F 1 "68k" H 11600 1250 50  0000 C CNN
+F 2 "MATRIX_1.4:RESISTOR_AXIAL_0.5W" H 11750 1250 50  0001 C CNN
+F 3 "" H 11750 1250 50  0001 C CNN
+F 4 "0.5W" H 11600 1150 50  0000 C CNN "Wattage"
+	1    11750 1250
+	1    0    0    -1
+$EndComp
+$Comp
+L MATRIX_1.4:RESISTOR R614
+U 1 1 5CFF7D9B
+P 11750 6750
+F 0 "R614" H 11600 6850 50  0000 C CNN
+F 1 "68k" H 11600 6750 50  0000 C CNN
+F 2 "MATRIX_1.4:RESISTOR_AXIAL_0.5W" H 11750 6750 50  0001 C CNN
+F 3 "" H 11750 6750 50  0001 C CNN
+F 4 "0.5W" H 11600 6650 50  0000 C CNN "Wattage"
+	1    11750 6750
+	1    0    0    -1
+$EndComp
 $EndSCHEMATC

Commit message: Commit Wed May 15 21:01:56 UTC 2019
Parts:
- added R720: 100k, MATRIX_1.4:RESISTOR_AXIAL_0.5W, symbol MATRIX_1.4:RESISTOR
- added SR701: sw1 ON, MATRIX_1.4:RL-SLA24, symbol MATRIX_1.4:RELAY_STD
- R701: footprint MATRIX_1.4:RESISTOR_AXIAL_0.25W -> MATRIX_1.4:RESISTOR_AXIAL_0.5W; Wattage (none) -> 0.5W
Connections:
- net +RLC: now also SR701.3
- net -RLC: now also SR701.4
- net 0: now also R720.2
- net M_OUT: now also SR701.2; no longer L501.2
- new net: L501.2, R720.1, SR701.1
Other:
- note added: "To OUTPUT\nTERMINAL (+)"
- note removed: "To protector\nrelay +NC"
- note removed: "To protector\nrelay coil"
- moved on the sheet: D701
Changed lines of the file:
@@
 Sheet 1 1
 Title "1600W RMS Class-H Audio Power Amplifier Core Circuit"
-Date "2019-05-13"
+Date "2019-05-15"
 Rev ""
 Comp "Notice: LIMITER & F/S.O.C.P are courtesy of VCGA (https://github.com/vcga/vcga)"
@@
 Text GLabel 7050 6400 0    50   Input ~ 0
 -42V
-Text GLabel 15550 7900 2    50   Output ~ 0
+Text GLabel 15550 9300 2    50   Output ~ 0
 M_OUT
-Text HLabel 15700 4900 0    50   BiDi ~ 0
+Text HLabel 15450 9150 2    50   BiDi ~ 0
 M_OUT
 Text HLabel 7800 800  0    50   BiDi ~ 0
@@
 $EndComp
 Wire Wire Line
-	14800 8850 14800 8800
-Wire Wire Line
 	14800 9600 14800 9650
-Wire Wire Line
-	14800 8800 14950 8800
-Connection ~ 14800 8800
-Wire Wire Line
-	14800 8800 14800 8650
-Text GLabel 14950 8800 2    50   Output ~ 0
-+RLC
-Text GLabel 14950 9100 2    50   Output ~ 0
--RLC
 Text HLabel 14950 9250 2    50   BiDi ~ 0
 -RLC
@@
 +RLC
 Wire Wire Line
-	14800 9050 14800 9100
-Wire Wire Line
-	14800 9100 14800 9250
-Connection ~ 14800 9100
-Wire Wire Line
-	14800 9100 14950 9100
-Wire Wire Line
 	14950 8650 14800 8650
 Connection ~ 14800 8650
@@
 	0    -1   -1   0
 $EndComp
-Text Notes 15350 9000 0    50   ~ 0
-To protector\nrelay coil
-Wire Notes Line
-	15300 8800 15300 9050
-Wire Notes Line
-	15300 9050 15850 9050
-Wire Notes Line
-	15850 9050 15850 8800
-Wire Notes Line
-	15850 8800 15300 8800
 $Comp
 L MATRIX_1.4:JRC4558 XU701
@@
 Wire Wire Line
 	8750 9450 8750 9400
-$Comp
-L MATRIX_1.4:RESISTOR R701
-U 1 1 6F7AF933
-P 8600 8250
-F 0 "R701" H 8350 8300 50  0000 L CNN
-F 1 "100k" H 8350 8200 50  0000 L CNN
-F 2 "MATRIX_1.4:RESISTOR_AXIAL_0.25W" H 8600 8250 50  0001 C CNN
-F 3 "" H 8600 8250 50  0001 C CNN
-	1    8600 8250
-	1    0    0    -1
-$EndComp
 Wire Wire Line
 	8800 8450 8600 8450
@@
 Text GLabel 14200 1750 2    50   BiDi ~ 0
 M_VSWON
-Text Notes 15350 8200 0    50   ~ 0
-To protector\nrelay +NC
+Text Notes 15300 9600 0    50   ~ 0
+To OUTPUT\nTERMINAL (+)
 Wire Notes Line
-	15300 8000 15300 8250
+	15250 9400 15250 9650
 Wire Notes Line
-	15300 8250 15850 8250
+	15250 9650 15850 9650
 Wire Notes Line
-	15850 8250 15850 8000
+	15850 9650 15850 9400
 Wire Notes Line
-	15850 8000 15300 8000
+	15850 9400 15250 9400
 $Comp
 L MATRIX_1.4:RESISTOR R520
@@
 	15750 4000 15800 4000
 Wire Wire Line
-	15800 4000 15800 4900
-Wire Wire Line
-	8600 8450 8600 9150
+	8600 8450 8600 8650
 Connection ~ 8600 8450
 $Comp
 L MATRIX_1.4:DIODE D701
 U 1 1 5DC31476
-P 8400 8450
-F 0 "D701" V 8250 8450 50  0000 C CNN
-F 1 "1N4148" V 8150 8450 50  0000 C CNN
-F 2 "MATRIX_1.4:DIODE_AXIAL_SMALL_GE" H 9400 8200 50  0001 C CNN
-F 3 "" H 8400 8450 50  0001 C CNN
-F 4 "D" H 9350 8400 50  0001 C CNN "Spice_Primitive"
-F 5 "1N4148" H 9350 8500 50  0001 C CNN "Spice_Model"
-F 6 "Y" H 9350 8300 50  0001 C CNN "Spice_Netlist_Enabled"
-F 7 "spice_models/model.lib" H 9350 8600 50  0001 C CNN "Spice_Lib_File"
-	1    8400 8450
+P 8400 8650
+F 0 "D701" V 8250 8650 50  0000 C CNN
+F 1 "1N4148" V 8150 8650 50  0000 C CNN
+F 2 "MATRIX_1.4:DIODE_AXIAL_SMALL_GE" H 9400 8400 50  0001 C CNN
+F 3 "" H 8400 8650 50  0001 C CNN
+F 4 "D" H 9350 8600 50  0001 C CNN "Spice_Primitive"
+F 5 "1N4148" H 9350 8700 50  0001 C CNN "Spice_Model"
+F 6 "Y" H 9350 8500 50  0001 C CNN "Spice_Netlist_Enabled"
+F 7 "spice_models/model.lib" H 9350 8800 50  0001 C CNN "Spice_Lib_File"
+	1    8400 8650
 	0    -1   -1   0
 $EndComp
@@
 L pspice:0 #GND0132
 U 1 1 5DC37366
-P 8200 8800
-F 0 "#GND0132" H 8200 8700 50  0001 C CNN
-F 1 "0" H 8200 8887 50  0001 C CNN
-F 2 "" H 8200 8800 50  0001 C CNN
-F 3 "~" H 8200 8800 50  0001 C CNN
-	1    8200 8800
+P 8200 9000
+F 0 "#GND0132" H 8200 8900 50  0001 C CNN
+F 1 "0" H 8200 9087 50  0001 C CNN
+F 2 "" H 8200 9000 50  0001 C CNN
+F 3 "~" H 8200 9000 50  0001 C CNN
+	1    8200 9000
 	1    0    0    -1
 $EndComp
 Wire Wire Line
-	8200 8800 8200 8450
+	8200 9000 8200 8650
 Wire Wire Line
-	8200 8450 8300 8450
-Wire Wire Line
-	8500 8450 8600 8450
+	8200 8650 8300 8650
 Wire Wire Line
 	8600 9450 8600 9350
@@
 	15150 4000 15300 4000
 Wire Wire Line
-	15800 4900 15700 4900
-Wire Wire Line
-	15800 4900 15800 7650
-Wire Wire Line
-	15800 7650 15400 7650
-Wire Wire Line
-	15400 7650 15400 7900
-Wire Wire Line
-	15400 7900 15550 7900
-Connection ~ 15800 4900
-Wire Wire Line
 	15000 7650 12450 7650
 Wire Wire Line
@@
 	1    0    0    -1
 $EndComp
+Wire Wire Line
+	14800 9050 14800 9150
+Wire Wire Line
+	14800 8650 14800 8750
+$Comp
+L MATRIX_1.4:RELAY_STD SR701
+U 1 1 5D1450E9
+P 15200 8950
+F 0 "SR701" H 15500 8950 50  0000 L CNN
+F 1 "sw1 ON" H 15480 8912 40  0001 L CNN
+F 2 "MATRIX_1.4:RL-SLA24" H 15200 8950 40  0001 C CNN
+F 3 "" H 15200 8950 40  0001 C CNN
+F 4 "SLA-24VDC-S L-C" H 15350 9100 40  0000 L CNB "Specification"
+	1    15200 8950
+	1    0    0    -1
+$EndComp
+Wire Wire Line
+	14800 8750 15100 8750
+Wire Wire Line
+	15100 8750 15100 8800
+Connection ~ 14800 8750
+Wire Wire Line
+	14800 8750 14800 8850
+Wire Wire Line
+	15100 9100 15100 9150
+Wire Wire Line
+	15100 9150 14800 9150
+Connection ~ 14800 9150
+Wire Wire Line
+	14800 9150 14800 9250
+Wire Wire Line
+	15300 9100 15300 9150
+Wire Wire Line
+	15300 9300 15550 9300
+Wire Wire Line
+	15800 8050 15600 8050
+Wire Wire Line
+	15300 8050 15300 8800
+Wire Wire Line
+	15800 4000 15800 8050
+Wire Wire Line
+	15450 9150 15300 9150
+Connection ~ 15300 9150
+Wire Wire Line
+	15300 9150 15300 9300
+$Comp
+L MATRIX_1.4:RESISTOR R701
+U 1 1 5CEFF2B0
+P 8600 8250
+F 0 "R701" H 8450 8350 50  0000 C CNN
+F 1 "100k" H 8450 8250 50  0000 C CNN
+F 2 "MATRIX_1.4:RESISTOR_AXIAL_0.5W" H 8600 8250 50  0001 C CNN
+F 3 "" H 8600 8250 50  0001 C CNN
+F 4 "0.5W" H 8450 8150 50  0000 C CNN "Wattage"
+	1    8600 8250
+	1    0    0    -1
+$EndComp
+Wire Wire Line
+	8500 8650 8600 8650
+Connection ~ 8600 8650
+Wire Wire Line
+	8600 8650 8600 9150
+$Comp
+L MATRIX_1.4:RESISTOR R720
+U 1 1 5D1551E5
+P 15600 8250
+F 0 "R720" H 15450 8350 50  0000 C CNN
+F 1 "100k" H 15450 8250 50  0000 C CNN
+F 2 "MATRIX_1.4:RESISTOR_AXIAL_0.5W" H 15600 8250 50  0001 C CNN
+F 3 "" H 15600 8250 50  0001 C CNN
+F 4 "0.5W" H 15450 8150 50  0000 C CNN "Wattage"
+	1    15600 8250
+	1    0    0    -1
+$EndComp
+$Comp
+L pspice:0 #GND?
+U 1 1 5D1579E4
+P 15600 8450
+F 0 "#GND?" H 15600 8350 50  0001 C CNN
+F 1 "0" H 15600 8537 50  0001 C CNN
+F 2 "" H 15600 8450 50  0001 C CNN
+F 3 "~" H 15600 8450 50  0001 C CNN
+	1    15600 8450
+	1    0    0    -1
+$EndComp
+Wire Wire Line
+	15600 8100 15600 8050
+Connection ~ 15600 8050
+Wire Wire Line
+	15600 8050 15300 8050
+Wire Wire Line
+	15600 8400 15600 8450
 $EndSCHEMATC
