File: schematics/1600WRMS-MATRIX-1.4-III-CLASS-H-AUDIO-POWER-AMPLIFIER-NS-LAB-VERSION/1600WRMS-MATRIX-1.4-III-CLASS-H-AUDIO-POWER-AMPLIFIER-NS-LAB-VERSION.kicad_pcb (KiCad board)
At the start: 2 copper layers, 267 parts, among them Q301 2N5551, Q401 2N5551, Q402 2N5551, Q403 2N5551, Q404 MJE340, Q405 MJE350, Q406 MJE350, Q407 MJE350, Q408 2N5551, Q409 MJE340, Q501 2N5401, Q502 MJE350, Q503 2N5551, Q504 MJE340, Q505 MJE340, Q506 MJE15032, Q507 2SC5200, Q5081 2SC5200, Q50810 2SC5200, Q50811 2SC5200, Q5082 2SC5200, Q5083 2SC5200, Q5084 2SC5200, Q5085 2SC5200, Q5086 2SC5200, Q5087 2SC5200, Q5088 2SC5200, Q5089 2SC5200, Q509 MJE15033, Q510 2SA1943, Q511 2SA1943, Q5111 2SA1943, Q51110 2SA1943, Q51111 2SA1943, Q5113 2SA1943, Q5114 2SA1943, Q5115 2SA1943, Q5116 2SA1943, Q5117 2SA1943, Q5118 2SA1943, Q5119 2SA1943, Q512 2N5551, Q513 2N5401, Q601 2N5551, Q602 2N5401, Q603 2N5401, Q604 2N5401, Q605 2N5551, Q606 2N5551, Q701 2N5551, Q702 2N5401, Q703 2N5551, Q704 2N5551, Q705 TIP42C, X6011 IRF9540, X6012 IRF9540, X6021 IRF540, X6022 IRF540

Commit message: Commit Thu May  9 01:23:26 UTC 2019
Parts:
- removed D401: 1N4004, MATRIX_1.4:DIODE_AXIAL_SMALL_SI
- removed R4051, R4061: 470, MATRIX_1.4:RESISTOR_AXIAL_0.25W
- removed R4052, R4062: 22, MATRIX_1.4:RESISTOR_AXIAL_0.25W
- removed R409: 270, MATRIX_1.4:RESISTOR_AXIAL_0.25W
- removed R4111, R4151: 150, MATRIX_1.4:RESISTOR_AXIAL_0.25W
- removed R4112: 680, MATRIX_1.4:RESISTOR_AXIAL_0.25W
- removed R414: 22k, MATRIX_1.4:RESISTOR_AXIAL_2W
- removed R4152: 750, MATRIX_1.4:RESISTOR_AXIAL_0.25W
- removed the R619 at (173.4, 66.4)
- removed the R619 at (270.3, 104.5)
- removed XRV401: VR, MATRIX_1.4:RESISTOR_ROUND_TRIMPOT_STD
- added Q410: MJE340, MATRIX_1.4:TO-225, F.Cu at (167.0, 154.4)
- added R405: 470, MATRIX_1.4:RESISTOR_AXIAL_0.25W, F.Cu at (144.9, 129.9)
- added R406: 470, MATRIX_1.4:RESISTOR_AXIAL_0.25W, F.Cu at (132.7, 142.2)
- added R4091: 150, MATRIX_1.4:RESISTOR_AXIAL_0.25W, F.Cu at (119.0, 141.0)
- added R4092: 680, MATRIX_1.4:RESISTOR_AXIAL_0.25W, F.Cu at (245.1, 26.9)
- added R411: 22k, MATRIX_1.4:RESISTOR_AXIAL_2W, F.Cu at (161.7, 40.7)
- added R4141: 150, MATRIX_1.4:RESISTOR_AXIAL_0.25W, F.Cu at (180.5, 110.4)
- added R4142: 750, MATRIX_1.4:RESISTOR_AXIAL_0.25W, F.Cu at (180.5, 114.5)
- added R619: 47k, MATRIX_1.4:RESISTOR_AXIAL_0.5W, F.Cu at (86.9, 144.9)
- D301, D302: value 1N4738 -> 1N4730
- Q403: value 2N5551 -> 2N5401
- Q404: value MJE340 -> 2N5401; footprint MATRIX_1.4:TO-225 -> MATRIX_1.4:TO-92-EBC
- Q405: value MJE350 -> 2N5551; footprint MATRIX_1.4:TO-225 -> MATRIX_1.4:TO-92-EBC
- Q406: value MJE350 -> MJE340
- Q407: value MJE350 -> 2N5401; footprint MATRIX_1.4:TO-225 -> MATRIX_1.4:TO-92-EBC
- Q408: value 2N5551 -> MJE350; footprint MATRIX_1.4:TO-92-EBC -> MATRIX_1.4:TO-225
- Q409: value MJE340 -> MJE350
- R4011, R4041: value 300 -> 270
- R4012, R4042: value 4.7k -> 150k
- R407: value 5.6k -> 270
- R408: value 5.6k -> 22k; footprint MATRIX_1.4:RESISTOR_AXIAL_0.25W -> MATRIX_1.4:RESISTOR_AXIAL_2W
- R410: value 22k -> 270; footprint MATRIX_1.4:RESISTOR_AXIAL_2W -> MATRIX_1.4:RESISTOR_AXIAL_0.25W
- R4122: value 750 -> 680
- moved R719 215.7 mm to (44.5, 155.0)
- moved R307 215.7 mm to (64.6, 155.0)
- moved D620 176.2 mm to (230.3, 26.8)
- moved R718 175.5 mm to (156.1, 98.2)
- moved R402 174.2 mm to (258.8, 26.9)
- moved Q705 170.0 mm to (156.6, 155.4)
- moved D304 169.0 mm to (101.6, 153.4)
- moved D302 167.4 mm to (85.7, 153.4)
- moved R710 159.7 mm to (129.1, 134.0)
- moved D704 156.0 mm to (132.7, 121.9)
- moved R712 154.6 mm to (163.7, 114.6)
- moved C302 154.5 mm to (172.9, 145.7)
- moved R304 154.4 mm to (130.1, 150.3)
- moved Q703 151.6 mm to (183.1, 149.0)
- moved R5145 149.7 mm to (246.1, 39.2)
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Connections:
- C301 pad 1: M_INPUT -> (no net)
- C402 pad 2: /M_REF -> Net-(C402-Pad2)
- C404 pad 2: /M_VASOUT -> Net-(C404-Pad2)
- C405 pad 2: /M_VASIOUT -> Net-(C404-Pad2)
- D503 pad 2: /M_VASOUT -> Net-(C404-Pad2)
- D504 pad 1: /M_VASOUT -> Net-(C404-Pad2)
- L501 pad 2: M_OUT -> (no net)
- Q401 pad 2: /M_REF -> Net-(C402-Pad2)
- Q402 pad 1: Net-(C405-Pad1) -> +120V
- Q402 pad 2: /M_NFB -> Net-(Q402-Pad2)
- Q403 pad 1: Net-(Q403-Pad1) -> Net-(C405-Pad1)
- Q403 pad 2: Net-(Q403-Pad2) -> Net-(C402-Pad2)
- Q403 pad 3: -120V -> Net-(Q403-Pad3)
- Q404 pad 1: Net-(Q404-Pad1) -> -120V
- Q404 pad 2: Net-(Q403-Pad1) -> Net-(Q402-Pad2)
- Q404 pad 3: Net-(Q403-Pad2) -> Net-(Q403-Pad3)
- Q405 pad 1: /M_VASOUT -> Net-(Q405-Pad1)
- Q405 pad 2: Net-(C404-Pad1) -> Net-(Q405-Pad2)
- Q405 pad 3: Net-(Q405-Pad3) -> -120V
- Q406 pad 1: /M_VASIOUT -> Net-(Q406-Pad1)
- Q406 pad 2: Net-(C405-Pad1) -> Net-(Q405-Pad1)
- Q406 pad 3: Net-(Q406-Pad3) -> Net-(Q405-Pad2)
- Q407 pad 2: Net-(D401-Pad2) -> Net-(Q407-Pad2)
- Q407 pad 3: /M_VASIOUT -> +120V
- Q408 pad 1: Net-(Q407-Pad1) -> Net-(Q408-Pad1)
- Q408 pad 2: Net-(Q408-Pad2) -> Net-(Q407-Pad1)
- Q408 pad 3: -120V -> Net-(Q407-Pad2)
- Q409 pad 1: /M_VASOUT -> Net-(C404-Pad2)
- Q409 pad 2: Net-(Q407-Pad1) -> Net-(C404-Pad1)
- Q409 pad 3: Net-(Q408-Pad2) -> Net-(Q409-Pad3)
- R4011 pad 2: /M_REF -> Net-(C402-Pad2)
- R4012 pad 2: /M_REF -> Net-(C402-Pad2)
- R402 pad 1: /M_REF -> Net-(C402-Pad2)
- R403 pad 2: /M_NFB -> Net-(Q402-Pad2)
- R4041 pad 2: /M_NFB -> Net-(Q402-Pad2)
- R4042 pad 2: /M_NFB -> Net-(Q402-Pad2)
- R407 pad 1: Net-(R407-Pad1) -> Net-(Q401-Pad3)
- R407 pad 2: Net-(C404-Pad1) -> Net-(Q406-Pad1)
- R408 pad 1: Net-(R408-Pad1) -> 0
- R408 pad 2: Net-(C405-Pad1) -> Net-(Q405-Pad1)
- R410 pad 1: 0 -> Net-(Q408-Pad1)
- R410 pad 2: Net-(Q403-Pad1) -> Net-(Q403-Pad3)
- R4121 pad 2: Net-(Q405-Pad3) -> Net-(Q407-Pad2)
- R4122 pad 2: Net-(Q405-Pad3) -> Net-(Q407-Pad2)
- R4131 pad 2: Net-(Q406-Pad3) -> Net-(Q409-Pad3)
- R4132 pad 2: Net-(Q406-Pad3) -> Net-(Q409-Pad3)

Commit message: Commit Thu May  9 10:32:49 UTC 2019
Parts:
- added R305: 100k, MATRIX_1.4:RESISTOR_AXIAL_0.5W, F.Cu at (238.8, 130.6)
- added R310: 2.7k, MATRIX_1.4:RESISTOR_AXIAL_0.25W, F.Cu at (236.2, 135.4)
- C302: value 220uF -> 10uF
- D301, D302: value 1N4730 -> 1N4734
- R4012, R4042: value 150k -> 2.0
- moved R4042 101.2 mm to (250.0, 135.4)
- moved R4011 85.0 mm to (236.2, 139.5)
- renumbered R305 to R309, R309 to R311, R310 to R312, R311 to R313, R312 to R314
Connections:
- R309 pad 2: Net-(R305-Pad2) -> Net-(R309-Pad2)
- R4011 pad 2: Net-(C402-Pad2) -> Net-(R4011-Pad2)
- R4012 pad 1: Net-(C401-Pad2) -> Net-(R4011-Pad2)
- R4041 pad 1: Net-(C403-Pad1) -> Net-(R4041-Pad1)
- R4042 pad 1: Net-(C403-Pad1) -> Net-(R4041-Pad1)
- R4042 pad 2: Net-(Q402-Pad2) -> Net-(C403-Pad1)
- XU302 pad 3: Net-(R305-Pad2) -> Net-(R309-Pad2)

Commit message: Commit Thu May  9 11:45:40 UTC 2019
Parts:
- C302: value 10uF -> 220uF
Changed lines of the file:
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@@
       (effects (font (size 1.27 1.27) (thickness 0.254)))
     )
-    (fp_text value 10uF (at 0 6.35) (layer F.Fab)
+    (fp_text value 220uF (at 0 6.35) (layer F.Fab)
       (effects (font (size 1.27 1.27) (thickness 0.254)))
     )

Commit message: Commit Mon May 13 03:44:39 UTC 2019
Parts:
- R605, R614: footprint MATRIX_1.4:RESISTOR_AXIAL_0.25W -> MATRIX_1.4:RESISTOR_AXIAL_0.5W
- X6011, X6012, X6021, X6022: footprint MATRIX_1.4:TO-220 -> MATRIX_1.4:TO-220-MIRRORED
- moved R614 99.2 mm to (235.0, 151.4)
- moved R605 83.1 mm to (235.0, 145.8)
- renumbered Q511 to Q5112

Commit message: Commit Wed May 15 21:01:56 UTC 2019
Parts:
- added R720: 100k, MATRIX_1.4:RESISTOR_AXIAL_0.5W, F.Cu at (283.2, 87.9)
- added SR701: sw1 ON, MATRIX_1.4:RL-SLA24, F.Cu at (298.4, 110.5)
- R701: footprint MATRIX_1.4:RESISTOR_AXIAL_0.25W -> MATRIX_1.4:RESISTOR_AXIAL_0.5W
- moved R701 62.1 mm to (283.2, 82.3)
Connections:
- net +RLC renamed /+RLC
- net -RLC renamed /-RLC
- L501 pad 2: (no net) -> Net-(L501-Pad2)
